Commit message: getting error about invalid kinematics parameter file

File: my_robot_cell/my_robot_cell_control/urdf/my_robot_cell_controlled.urdf.xacro (robot description, xacro)
@@ -4,11 +4,13 @@
   <xacro:include filename="$(find my_robot_cell_description)/urdf/my_robot_cell_macro.xacro"/>
   <!--The driver already provides a control tag for the UR arm, we can directly include-->
-  <xacro:include filename="$(find ur_robot_driver)/urdf/ur.ros2_control.xacro"/>
+  <!-- I think this is what's giving me lots of issues... -->
+  <!-- <xacro:include filename="$(find ur_robot_driver)/urdf/ur.ros2_control.xacro"/> -->
+  <xacro:include filename="$(find ur_description)/urdf/ur.ros2_control.xacro"/>
   <!--We need to specify the arguments used for parametrizing our description-->
-  <xacro:arg name="ur_type" default="ur20"/>
+  <xacro:arg name="ur_type" default="ur5e"/>
   <xacro:arg name="joint_limit_parameters_file" default="$(find ur_description)/config/$(arg ur_type)/joint_limits.yaml"/>
-  <xacro:arg name="kinematics_parameters_file" default="$(find ur_description)/config/$(arg ur_type)/default_kinematics.yaml"/>
   <xacro:arg name="physical_parameters_file" default="$(find ur_description)/config/$(arg ur_type)/physical_parameters.yaml"/>
   <xacro:arg name="visual_parameters_file" default="$(find ur_description)/config/$(arg ur_type)/visual_parameters.yaml"/>
+  <xacro:arg name="kinematics_parameters_file" default="$(find ur_description)/config/$(arg ur_type)/default_kinematics.yaml"/>
   <xacro:arg name="robot_ip" default="0.0.0.0"/>
   <xacro:arg name="headless_mode" default="false" />
@@ -20,4 +22,5 @@
   <link name="world" />
   <!--Create the scene description including the robot-->
+  <!-- this hsould include the table, and end effector aswell! -->
   <xacro:my_robot_cell
     parent="world"
@@ -31,4 +34,5 @@
   </xacro:my_robot_cell>
   <!--Create the control tag for the UR robot-->
+  <!-- This is failing at the kinematics portion-->
   <xacro:ur_ros2_control
     name="$(arg ur_type)"

File: my_robot_cell/my_robot_cell_description/urdf/my_robot_cell.urdf.xacro (robot description, xacro)
@@ -2,5 +2,5 @@
 <robot name="my_robot_cell" xmlns:xacro="http://ros.org/wiki/xacro">
   <xacro:include filename="$(find my_robot_cell_description)/urdf/my_robot_cell_macro.xacro"/>
-  <xacro:arg name="ur_type" default="ur20"/>
+  <xacro:arg name="ur_type" default="ur5e"/>
   <xacro:arg name="joint_limits_parameters_file" default="$(find ur_description)/config/$(arg ur_type)/joint_limits.yaml"/>
   <xacro:arg name="kinematics_parameters_file" default="$(find ur_description)/config/$(arg ur_type)/default_kinematics.yaml"/>

File: my_robot_cell/my_robot_cell_description/urdf/my_robot_cell_macro.xacro (robot description, xacro)
@@ -1,4 +1,5 @@
 <?xml version="1.0"?>
 <robot xmlns:xacro="http://ros.org/wiki/xacro">
+  <!-- Include the true and honest robot from UR's code -->
   <xacro:include filename="$(find ur_description)/urdf/ur_macro.xacro"/>
   <xacro:macro name="my_robot_cell" params="
@@ -11,4 +12,5 @@
     visual_parameters_file
     ">
+    <!-- connects world(?) to table -->
     <joint name="table_base_joint" type="fixed">
       <xacro:insert_block name="origin" />
@@ -16,62 +18,32 @@
       <child link="table" />
     </joint>
+    <!-- The table the robot sits on -->
     <link name="table">
       <visual>
         <geometry>
-          <mesh filename="package://my_robot_cell_description/meshes/fzi_table.dae"/>
+          <box size="1 2 0.05"/>
         </geometry>
-        <origin rpy="0 0 0" xyz="0.75 0.5 -1"/>
+        <origin xyz="-0.5 0 -0.025" rpy="0 0 0"/>
+        <material name="white">
+          <color rgba="1 1 1 1"/>
+        </material>
       </visual>
       <collision>
         <geometry>
-          <mesh filename="package://my_robot_cell_description/meshes/fzi_table.dae"/>
+          <box size="1 2 0.05"/>
         </geometry>
-        <origin rpy="0 0 0" xyz="0.75 0.5 -1"/>
+        <!-- TODO, measure how thick and how far in on the real table the mounting plate is-->
+        <origin xyz="-0.5 0 -0.020" rpy="0 0 0"/>
       </collision>
     </link>
-    <link name="monitor">
-      <visual>
-        <geometry>
-          <mesh filename="package://my_robot_cell_description/meshes/171005_Motek_Monitor_L.dae"/>
-        </geometry>
-      </visual>
-      <collision>
-        <geometry>
-          <mesh filename="package://my_robot_cell_description/meshes/171005_Motek_Monitor_L.dae"/>
-        </geometry>
-      </collision>
-    </link>
-    <joint name="base_to_monitor" type="fixed">
-      <parent link="table"/>
-      <child link="monitor"/>
-      <origin xyz="0.2 0.6 0"/>
-    </joint>
-    <material name="white">
-      <color rgba="1 1 1 1"/>
-    </material>
-    <link name="wall">
-      <visual>
-        <geometry>
-          <mesh filename="package://my_robot_cell_description/meshes/wall.dae"/>
-        </geometry>
-      </visual>
-      <collision>
-        <geometry>
-          <box size="4.44 0.1 2.5"/>
-        </geometry>
-      </collision>
-    </link>
-    <joint name="base_to_wall" type="fixed">
-      <parent link="table"/>
-      <child link="wall"/>
-      <origin xyz="1.25 1.5 0.5"/>
-    </joint>
-    <link name="robot_mount"/>
     <joint name="base_to_robot_mount" type="fixed">
       <parent link="table"/>
       <child link="robot_mount"/>
-      <origin xyz="0.845 0.85 0" rpy="0 0 ${pi}" />
+      <origin xyz="-0.15 0 0.025" rpy="0 0 ${pi}" />
     </joint>
-    <!--This will create the specific robot-->
+    <!-- Link that joins OUR stuff, to the robot -->
+    <link name="robot_mount"/>
+    <!--This will create the specific robot -->
+    <!-- Call UR's code for making the true and honest robot arm" -->
     <xacro:ur_robot
       name="${ur_type}"
@@ -82,7 +54,31 @@
       physical_parameters_file="${physical_parameters_file}"
       visual_parameters_file="${visual_parameters_file}"
+      generate_ros2_control_tag="false"
     >
       <origin xyz="0 0 0" rpy="0 0 0" />
     </xacro:ur_robot>
+    <!-- End effector -->
+    <joint name="tool0_to_end_effector" type="fixed">
+        <parent link="${ur_type}_tool0"/>
+        <child link="end_effector"/>
+        <origin xyz="0 0 0"/>
+    </joint>
+    <link name="end_effector">
+        <visual>
+            <material name="blue">
+              <color rgba="0 0.7 1 1"/>
+            </material>
+            <geometry>
+                <cylinder length="0.125" radius="0.0125"/>
+            </geometry>
+            <origin xyz="0 0 0.0625"/>
+        </visual>
+        <collision>
+            <geometry>
+                <cylinder length="0.125" radius="0.0125"/>
+            </geometry>
+            <origin xyz="0 0 0.0625"/>
+        </collision>
+    </link>
   </xacro:macro>
 </robot>
