Commit message: changed to have visual be the ur5

File: my_robot_cell/my_robot_cell_description/urdf/my_robot_cell_macro.xacro (robot description, xacro)
@@ -1,4 +1,5 @@
 <?xml version="1.0"?>
 <robot xmlns:xacro="http://ros.org/wiki/xacro">
+  <!-- Include the true and honest robot from UR's code -->
   <xacro:include filename="$(find ur_description)/urdf/ur_macro.xacro"/>
   <xacro:macro name="my_robot_cell" params="
@@ -11,4 +12,5 @@
     visual_parameters_file
     ">
+    <!-- connects world(?) to table -->
     <joint name="table_base_joint" type="fixed">
       <xacro:insert_block name="origin" />
@@ -16,62 +18,32 @@
       <child link="table" />
     </joint>
+    <!-- The table the robot sits on -->
     <link name="table">
       <visual>
         <geometry>
-          <mesh filename="package://my_robot_cell_description/meshes/fzi_table.dae"/>
+          <box size="1 2 0.05"/>
         </geometry>
-        <origin rpy="0 0 0" xyz="0.75 0.5 -1"/>
+        <origin xyz="-0.5 0 -0.025" rpy="0 0 0"/>
+        <material name="white">
+          <color rgba="1 1 1 1"/>
+        </material>
       </visual>
       <collision>
         <geometry>
-          <mesh filename="package://my_robot_cell_description/meshes/fzi_table.dae"/>
+          <box size="1 2 0.05"/>
         </geometry>
-        <origin rpy="0 0 0" xyz="0.75 0.5 -1"/>
+        <!-- TODO, measure how thick and how far in on the real table the mounting plate is-->
+        <origin xyz="-0.5 0 -0.020" rpy="0 0 0"/>
       </collision>
     </link>
-    <link name="monitor">
-      <visual>
-        <geometry>
-          <mesh filename="package://my_robot_cell_description/meshes/171005_Motek_Monitor_L.dae"/>
-        </geometry>
-      </visual>
-      <collision>
-        <geometry>
-          <mesh filename="package://my_robot_cell_description/meshes/171005_Motek_Monitor_L.dae"/>
-        </geometry>
-      </collision>
-    </link>
-    <joint name="base_to_monitor" type="fixed">
-      <parent link="table"/>
-      <child link="monitor"/>
-      <origin xyz="0.2 0.6 0"/>
-    </joint>
-    <material name="white">
-      <color rgba="1 1 1 1"/>
-    </material>
-    <link name="wall">
-      <visual>
-        <geometry>
-          <mesh filename="package://my_robot_cell_description/meshes/wall.dae"/>
-        </geometry>
-      </visual>
-      <collision>
-        <geometry>
-          <box size="4.44 0.1 2.5"/>
-        </geometry>
-      </collision>
-    </link>
-    <joint name="base_to_wall" type="fixed">
-      <parent link="table"/>
-      <child link="wall"/>
-      <origin xyz="1.25 1.5 0.5"/>
-    </joint>
-    <link name="robot_mount"/>
     <joint name="base_to_robot_mount" type="fixed">
       <parent link="table"/>
       <child link="robot_mount"/>
-      <origin xyz="0.845 0.85 0" rpy="0 0 ${pi}" />
+      <origin xyz="-0.15 0 0.025" rpy="0 0 ${pi}" />
     </joint>
-    <!--This will create the specific robot-->
+    <!-- Link that joins OUR stuff, to the robot -->
+    <link name="robot_mount"/>
+    <!--This will create the specific robot -->
+    <!-- Call UR's code for making the true and honest robot arm" -->
     <xacro:ur_robot
       name="${ur_type}"
@@ -86,4 +58,27 @@
       <origin xyz="0 0 0" rpy="0 0 0" />
     </xacro:ur_robot>
+    <!-- End effector -->
+    <joint name="tool0_to_end_effector" type="fixed">
+        <parent link="${ur_type}_tool0"/>
+        <child link="end_effector"/>
+        <origin xyz="0 0 0"/>
+    </joint>
+    <link name="end_effector">
+        <visual>
+            <material name="blue">
+              <color rgba="0 0.7 1 1"/>
+            </material>
+            <geometry>
+                <cylinder length="0.125" radius="0.0125"/>
+            </geometry>
+            <origin xyz="0 0 0.0625"/>
+        </visual>
+        <collision>
+            <geometry>
+                <cylinder length="0.125" radius="0.0125"/>
+            </geometry>
+            <origin xyz="0 0 0.0625"/>
+        </collision>
+    </link>
   </xacro:macro>
 </robot>
